File: src/LED.kicad_pcb (KiCad board)
At the start: 2 copper layers, 10 x 10 mm, 9 parts, among them J1 Conn_01x03_Pin

Commit message: modified:   src/LED.kicad_pcb 	modified:   src/LED.kicad_pcb-bak 	modified:   src/LED.kicad_sch 	modified:   src/LED.xml 	modified:   src/LED_s.kicad_sch
Other:
- board text added: "0.2 mm"
- board text added: "0.2 mm / 0.15 mm"
- board text added: "1.2 mm"
- board text added: "10 mm x 10 mm"
- board text removed: "0.2000 mm"
- board text removed: "0.2000 mm / 0.1500 mm"
- board text removed: "1.2000 mm"
- board text removed: "10.0000 mm x 10.0000 mm"
Changed lines of the file:
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@@
 	(title_block
 		(title "LED")
-		(date "%%date%%")
+		(date "2026-07-03 23:14:13")
 		(rev "bdd8a53")
 		(company "Engineering Services")
@@
 		)
 	)
-	(gr_text "0.2000 mm"
+	(gr_text "0.2 mm"
 		(at 111.649995 79.8 0)
 		(layer "Cmts.User")
@@
 		)
 	)
-	(gr_text "10.0000 mm x 10.0000 mm"
+	(gr_text "10 mm x 10 mm"
 		(at 52.55 75.843 0)
 		(layer "Cmts.User")
@@
 		)
 	)
-	(gr_text "0.2000 mm / 0.1500 mm"
+	(gr_text "0.2 mm / 0.15 mm"
 		(at 52.55 79.8 0)
 		(layer "Cmts.User")
@@
 		)
 	)
-	(gr_text "1.2000 mm"
+	(gr_text "1.2 mm"
 		(at 111.649995 71.886 0)
 		(layer "Cmts.User")

Commit message: improved fab layers
Parts:
- C1, C2, C3: value 1u -> 100n
- R1: value 500 -> 470
